File: hardware/rev1/jackboard/jackboard.sch (KiCad schematic (older format))
At the start: 12 parts, among them J1 AudioJack2_SwitchT, J10 AudioJack2_SwitchT, J11 USB_B, J2 Conn_01x10_Female, J3 Conn_01x10_Female, J4 AudioJack2_SwitchT, J5 AudioJack2_SwitchT, J6 AudioJack2_SwitchT, J7 AudioJack2_SwitchT, J8 AudioJack2_SwitchT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

Commit message: Wrap up prototype jackboard
Parts:
- added SW1: SW_Push, Button_Switch_THT:SW_PUSH_6mm, symbol Switch:SW_Push
Connections:
- net GND: now also SW1.2
- net Reset: now also SW1.1
Changed lines of the file:
@@
 EESchema Schematic File Version 4
-EELAYER 30 0
+LIBS:jackboard-cache
+EELAYER 29 0
 EELAYER END
 $Descr A4 11693 8268
@@
 	1    0    0    -1
 $EndComp
+$Comp
+L Switch:SW_Push SW1
+U 1 1 5E5DC434
+P 1500 4150
+F 0 "SW1" H 1500 4435 50  0000 C CNN
+F 1 "SW_Push" H 1500 4344 50  0000 C CNN
+F 2 "Button_Switch_THT:SW_PUSH_6mm" H 1500 4350 50  0001 C CNN
+F 3 "~" H 1500 4350 50  0001 C CNN
+	1    1500 4150
+	1    0    0    -1
+$EndComp
+Text GLabel 1300 4150 0    50   Input ~ 0
+Reset
+$Comp
+L power:GND #PWR0113
+U 1 1 5E5DD193
+P 1700 4150
+F 0 "#PWR0113" H 1700 3900 50  0001 C CNN
+F 1 "GND" V 1700 3950 50  0000 C CNN
+F 2 "" H 1700 4150 50  0001 C CNN
+F 3 "" H 1700 4150 50  0001 C CNN
+	1    1700 4150
+	0    -1   -1   0
+$EndComp
 $EndSCHEMATC
