File: hardware/rev1/mainboard/mainboard.kicad_pcb (KiCad board)
At the start: 2 copper layers, 40 x 108 mm, 59 parts, among them J1 CONN_05X2SHD, J2 Conn_01x10_Female, J3 Conn_01x10_Female, U1 LM1117-5.0, U2 TPS79633, U3 SAMD51J, U4 OPA388, U5 W25Q32FVSS, U6 AD5686xRUZ, U7 SN74AHCT125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

Commit message: Update all gerbes for latest PCB revisions
Parts:
- J1: footprint Connectors:2X5-SHROUDED -> SF Connectors:2X5-SHROUDED
- J2, J3: footprint Connectors:1X10_LOCK -> SF Connectors:1X10
Routing:
- net GND: vias 99 -> 95
Other:
- board text added: "Alethea Flowers CC-BY-SA 4.0 v6 2020/4/15 wntr.dev/sol"
- board text removed: "Alethea Flowers CC-BY-SA 4.0 v5 2020/1/15 wntr.dev"
