File: hardware/rev1/mainboard/mainboard.sch (KiCad schematic (older format))
At the start: 58 parts, among them J1 CONN_05X2SHD, J2 Conn_01x10_Female, J3 Conn_01x10_Female, U1 LM1117-5.0, U2 TPS79633, U3 SAMD51J, U4 OPA388, U5 W25Q32FVSS, U6 AD5686xRUZ, U7 SN74AHCT125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

Commit message: Assigning more MPNs
Parts:
- D1, D2: mpn 1N4148W -> 1N4148W-7-F
- R16, R17, R5, R7: mpn (none) -> ERA-8AEB2151V
- R2: mpn (none) -> ERA-8AEB112V
- R3: mpn (none) -> ERA8AEB102V
- U6: mpn AD5686RARUZ -> AD5686RBRUZ
Changed lines of the file:
@@
 F 2 "Diode_SMD:D_SOD-123" H 1650 1300 50  0001 C CNN
 F 3 "~" H 1650 1300 50  0001 C CNN
-F 4 "1N4148W" H 1650 1300 50  0001 C CNN "mpn"
+F 4 "1N4148W-7-F" H 1650 1300 50  0001 C CNN "mpn"
 	1    1650 1300
 	-1   0    0    1
@@
 F 2 "Resistor_SMD:R_1206_3216Metric_Pad1.42x1.75mm_HandSolder" V 2680 1100 50  0001 C CNN
 F 3 "~" H 2750 1100 50  0001 C CNN
+F 4 "ERA-8AEB112V" H 2750 1100 50  0001 C CNN "mpn"
 	1    2750 1100
 	1    0    0    -1
@@
 F 2 "Resistor_SMD:R_1206_3216Metric_Pad1.42x1.75mm_HandSolder" V 2680 1400 50  0001 C CNN
 F 3 "~" H 2750 1400 50  0001 C CNN
+F 4 "ERA8AEB102V" H 2750 1400 50  0001 C CNN "mpn"
 	1    2750 1400
 	1    0    0    -1
@@
 F 2 "Package_SO:TSSOP-16_4.4x5mm_P0.65mm" H 5000 1600 50  0001 C CNN
 F 3 "https://www.mouser.com/datasheet/2/609/AD5686R_5685R_5684R-1501714.pdf" H 5000 1600 50  0001 C CNN
-F 4 "AD5686RARUZ" H 5000 1600 50  0001 C CNN "mpn"
+F 4 "AD5686RBRUZ" H 5000 1600 50  0001 C CNN "mpn"
 	1    5000 1600
 	1    0    0    -1
@@
 F 2 "Resistor_SMD:R_1206_3216Metric_Pad1.42x1.75mm_HandSolder" V 6880 1550 50  0001 C CNN
 F 3 "~" H 6950 1550 50  0001 C CNN
+F 4 "ERA-8AEB2151V" H 6950 1550 50  0001 C CNN "mpn"
 	1    6950 1550
 	0    1    1    0
@@
 F 2 "Resistor_SMD:R_1206_3216Metric_Pad1.42x1.75mm_HandSolder" V 8780 1550 50  0001 C CNN
 F 3 "~" H 8850 1550 50  0001 C CNN
+F 4 "ERA-8AEB2151V" H 8850 1550 50  0001 C CNN "mpn"
 	1    8850 1550
 	0    1    1    0
@@
 F 2 "Resistor_SMD:R_1206_3216Metric_Pad1.42x1.75mm_HandSolder" V 6830 2350 50  0001 C CNN
 F 3 "~" H 6900 2350 50  0001 C CNN
+F 4 "ERA-8AEB2151V" H 6900 2350 50  0001 C CNN "mpn"
 	1    6900 2350
 	0    1    1    0
@@
 F 2 "Resistor_SMD:R_1206_3216Metric_Pad1.42x1.75mm_HandSolder" V 8730 2350 50  0001 C CNN
 F 3 "~" H 8800 2350 50  0001 C CNN
+F 4 "ERA-8AEB2151V" H 8800 2350 50  0001 C CNN "mpn"
 	1    8800 2350
 	0    1    1    0
@@
 F 2 "Diode_SMD:D_SOD-123" H 1650 900 50  0001 C CNN
 F 3 "~" H 1650 900 50  0001 C CNN
-F 4 "1N4148W" H 1650 900 50  0001 C CNN "mpn"
+F 4 "1N4148W-7-F" H 1650 900 50  0001 C CNN "mpn"
 	1    1650 900
 	1    0    0    -1

Commit message: Update all gerbes for latest PCB revisions
Parts:
- D1, D2: mpn 1N4148W-7-F -> MF-DIO-SOD123-1N4148
- J1: footprint Connectors:2X5-SHROUDED -> SF Connectors:2X5-SHROUDED; mpn (none) -> 61201021621
- J2, J3: footprint Connectors:1X10_LOCK -> SF Connectors:1X10; mpn (none) -> MF-CON-2.54mm-01x10
- R18, R19, R8, R9: mpn ERA8AEB9091V -> ERA8AEB912V
- U5: value W25Q32FVSS -> GD25Q64CSIGR; mpn W25Q32JVSSIQ TR -> GD25Q64CSIGR
Changed lines of the file:
@@
 EESchema Schematic File Version 4
-EELAYER 30 0
+LIBS:mainboard-cache
+EELAYER 29 0
 EELAYER END
 $Descr A4 11693 8268
@@
 Sheet 1 1
 Title "Sol Mainboard"
-Date "2020-01-05"
-Rev "Rev1 v1"
+Date "2020-04-15"
+Rev "Rev1 v2"
 Comp "Winterbloom"
 Comment1 "Alethea Flowers"
@@
 F 0 "J1" H 1250 1610 45  0000 C CNN
 F 1 "CONN_05X2SHD" H 1250 1526 45  0000 C CNN
-F 2 "Connectors:2X5-SHROUDED" H 1250 1500 20  0001 C CNN
+F 2 "SF Connectors:2X5-SHROUDED" H 1250 1500 20  0001 C CNN
 F 3 "" H 1250 1100 50  0001 C CNN
 F 4 "Eurorack Power" H 1250 1450 60  0000 C CNN "Field4"
 F 5 "https://www.sparkfun.com/products/8506" H 1250 1100 50  0001 C CNN "URL"
+F 6 "61201021621" H 1250 1100 50  0001 C CNN "mpn"
 	1    1250 1100
 	1    0    0    -1
@@
 F 2 "Diode_SMD:D_SOD-123" H 1650 1300 50  0001 C CNN
 F 3 "~" H 1650 1300 50  0001 C CNN
-F 4 "1N4148W-7-F" H 1650 1300 50  0001 C CNN "mpn"
+F 4 "MF-DIO-SOD123-1N4148" H 1650 1300 50  0001 C CNN "mpn"
 	1    1650 1300
 	-1   0    0    1
@@
 P 5975 4625
 F 0 "U5" H 5975 5135 45  0000 C CNN
-F 1 "W25Q32FVSS" H 5975 5051 45  0000 C CNN
+F 1 "GD25Q64CSIGR" H 5975 5051 45  0000 C CNN
 F 2 "flash:SOIC-8" H 5975 4975 20  0001 C CNN
 F 3 "" H 5975 4625 50  0001 C CNN
 F 4 "4MB QSPI Flash" H 5975 4956 60  0000 C CNN "Field4"
-F 5 "W25Q32JVSSIQ TR" H 5975 4625 50  0001 C CNN "mpn"
+F 5 "GD25Q64CSIGR" H 5975 4625 50  0001 C CNN "mpn"
 	1    5975 4625
 	1    0    0    -1
@@
 F 2 "Resistor_SMD:R_1206_3216Metric_Pad1.42x1.75mm_HandSolder" V 7530 1550 50  0001 C CNN
 F 3 "~" H 7600 1550 50  0001 C CNN
-F 4 "ERA8AEB9091V" H 7600 1550 50  0001 C CNN "mpn"
+F 4 "ERA8AEB912V" H 7600 1550 50  0001 C CNN "mpn"
 	1    7600 1550
 	0    1    1    0
@@
 F 2 "Resistor_SMD:R_1206_3216Metric_Pad1.42x1.75mm_HandSolder" V 9430 1550 50  0001 C CNN
 F 3 "~" H 9500 1550 50  0001 C CNN
-F 4 "ERA8AEB9091V" H 9500 1550 50  0001 C CNN "mpn"
+F 4 "ERA8AEB912V" H 9500 1550 50  0001 C CNN "mpn"
 	1    9500 1550
 	0    1    1    0
@@
 F 2 "Resistor_SMD:R_1206_3216Metric_Pad1.42x1.75mm_HandSolder" V 7480 2350 50  0001 C CNN
 F 3 "~" H 7550 2350 50  0001 C CNN
-F 4 "ERA8AEB9091V" H 7550 2350 50  0001 C CNN "mpn"
+F 4 "ERA8AEB912V" H 7550 2350 50  0001 C CNN "mpn"
 	1    7550 2350
 	0    1    1    0
@@
 F 2 "Resistor_SMD:R_1206_3216Metric_Pad1.42x1.75mm_HandSolder" V 9380 2350 50  0001 C CNN
 F 3 "~" H 9450 2350 50  0001 C CNN
-F 4 "ERA8AEB9091V" H 9450 2350 50  0001 C CNN "mpn"
+F 4 "ERA8AEB912V" H 9450 2350 50  0001 C CNN "mpn"
 	1    9450 2350
 	0    1    1    0
@@
 F 2 "Diode_SMD:D_SOD-123" H 1650 900 50  0001 C CNN
 F 3 "~" H 1650 900 50  0001 C CNN
-F 4 "1N4148W-7-F" H 1650 900 50  0001 C CNN "mpn"
+F 4 "MF-DIO-SOD123-1N4148" H 1650 900 50  0001 C CNN "mpn"
 	1    1650 900
 	1    0    0    -1
@@
 F 0 "J2" V 8790 3605 50  0000 C CNN
 F 1 "Conn_01x10_Female" V 8699 3605 50  0000 C CNN
-F 2 "Connectors:1X10_LOCK" H 8625 3675 50  0001 C CNN
+F 2 "SF Connectors:1X10" H 8625 3675 50  0001 C CNN
 F 3 "~" H 8625 3675 50  0001 C CNN
+F 4 "MF-CON-2.54mm-01x10" H 8625 3675 50  0001 C CNN "mpn"
 	1    8625 3675
 	0    -1   -1   0
@@
 F 0 "J3" V 10040 3605 50  0000 C CNN
 F 1 "Conn_01x10_Female" V 9949 3605 50  0000 C CNN
-F 2 "Connectors:1X10_LOCK" H 9875 3675 50  0001 C CNN
+F 2 "SF Connectors:1X10" H 9875 3675 50  0001 C CNN
 F 3 "~" H 9875 3675 50  0001 C CNN
+F 4 "MF-CON-2.54mm-01x10" H 9875 3675 50  0001 C CNN "mpn"
 	1    9875 3675
 	0    -1   -1   0
