File: hardware/rev1/mainboard/mainboard.sch (KiCad schematic (older format))
At the start: 58 parts, among them J1 CONN_05X2SHD, J2 Conn_01x10_Female, J3 Conn_01x10_Female, U1 LM1117-5.0, U2 TPS79633, U3 SAMD51J, U4 OPA388, U5 GD25Q64CSIGR, U6 AD5686xRUZ, U7 SN74AHCT125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

Commit message: Update PDF of schematic and add git pre-commit hook to make sure it stays up-to-date
Parts:
- J1: symbol SparkFun-Connectors:CONN_05X2SHD -> mainboard-rescue:CONN_05X2SHD-SparkFun-Connectors
Changed lines of the file:
@@
 EESchema Schematic File Version 4
-LIBS:mainboard-cache
-EELAYER 29 0
+EELAYER 30 0
 EELAYER END
 $Descr A4 11693 8268
@@
 $EndDescr
 $Comp
-L SparkFun-Connectors:CONN_05X2SHD J1
+L mainboard-rescue:CONN_05X2SHD-SparkFun-Connectors J1
 U 1 1 5D1D5204
 P 1250 1100
